File: neon-beat-buzzer-pcb.kicad_sch (KiCad schematic)
At the start: 62 parts, among them J1 BATT_CON, J2 SWITCH_CON, J3 BUTTON_CON, J4 USB_C_Receptacle_USB2.0_16P, U1 ESP32-C3-MINI-1, U2 BQ24074RGT, U3 TPS22929D, U4 74AHCT1G125, U5 TPS610997DRV, U6 USBLC6-2SC6, U7 XC6210B332MR

Commit message: project: partial routing
Signed-off-by: Alexis Lothoré <alexis.lothore@gmail.com>
Parts:
- removed R15: 0, Resistor_SMD:R_0805_2012Metric_Pad1.20x1.40mm_HandSolder, symbol Device:R
- added C17: 0.1uF, Capacitor_SMD:C_0805_2012Metric_Pad1.18x1.45mm_HandSolder, symbol Device:C
- C15, C16: footprint (none) -> Capacitor_SMD:C_0805_2012Metric_Pad1.18x1.45mm_HandSolder
- R16: footprint (none) -> Resistor_SMD:R_0805_2012Metric_Pad1.20x1.40mm_HandSolder
- U4: footprint (none) -> Package_TO_SOT_SMD:SOT-23-5
Connections:
- net GND: now also C17.2
- net v_5v: now also C17.1
- net v_batt_p: now also J1.1 (Pin_1)
- net at R3.1: now also U6.3 (I/O2); no longer U6.4 (I/O2)
- net at J4.A6 (D+), J4.B6 (D+): now also U6.4 (I/O2); no longer U6.3 (I/O2)
- net at J4.A7 (D-), J4.B7 (D-): now also U6.6 (I/O1); no longer U6.1 (I/O1)
- net at R4.1: now also U6.1 (I/O1); no longer U6.6 (I/O1)
Changed lines of the file:
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@@
 	)
 	(junction
+		(at 196.85 115.57)
+		(diameter 0)
+		(color 0 0 0 0)
+	)
+	(junction
 		(at 214.63 41.91)
 		(diameter 0)
@@
 	)
 	(junction
-		(at 53.34 175.26)
+		(at 191.77 106.68)
 		(diameter 0)
 		(color 0 0 0 0)
 	)
 	(junction
-		(at 209.55 125.73)
+		(at 53.34 175.26)
 		(diameter 0)
 		(color 0 0 0 0)
@@
 	(wire
 		(pts
-			(xy 26.67 170.18) (xy 29.21 170.18)
+			(xy 26.67 170.18) (xy 41.91 170.18)
 		)
 		(stroke
@@
 	(wire
 		(pts
-			(xy 124.46 104.14) (xy 124.46 113.03)
+			(xy 209.55 125.73) (xy 223.52 125.73)
 		)
 		(stroke
@@
 	(wire
 		(pts
-			(xy 195.58 125.73) (xy 209.55 125.73)
+			(xy 124.46 104.14) (xy 124.46 113.03)
 		)
 		(stroke
@@
 	(wire
 		(pts
+			(xy 191.77 106.68) (xy 196.85 106.68)
+		)
+		(stroke
+			(width 0)
+			(type default)
+		)
+	)
+	(wire
+		(pts
 			(xy 198.12 35.56) (xy 198.12 41.91)
 		)
@@
 	(wire
 		(pts
-			(xy 74.93 69.85) (xy 74.93 71.12)
+			(xy 196.85 114.3) (xy 196.85 115.57)
 		)
 		(stroke
@@
 	(wire
 		(pts
-			(xy 26.67 187.96) (xy 34.29 187.96)
+			(xy 74.93 69.85) (xy 74.93 71.12)
 		)
 		(stroke
@@
 	(wire
 		(pts
-			(xy 43.18 118.11) (xy 43.18 120.65)
+			(xy 26.67 187.96) (xy 34.29 187.96)
 		)
 		(stroke
@@
 	(wire
 		(pts
-			(xy 77.47 54.61) (xy 81.28 54.61)
+			(xy 43.18 118.11) (xy 43.18 120.65)
 		)
 		(stroke
@@
 	(wire
 		(pts
-			(xy 198.12 25.4) (xy 201.93 25.4)
+			(xy 77.47 54.61) (xy 81.28 54.61)
 		)
 		(stroke
@@
 	(wire
 		(pts
-			(xy 147.32 39.37) (xy 154.94 39.37)
+			(xy 198.12 25.4) (xy 201.93 25.4)
 		)
 		(stroke
@@
 	(wire
 		(pts
-			(xy 43.18 62.23) (xy 43.18 68.58)
+			(xy 147.32 39.37) (xy 154.94 39.37)
 		)
 		(stroke
@@
 	(wire
 		(pts
-			(xy 36.83 170.18) (xy 41.91 170.18)
+			(xy 43.18 62.23) (xy 43.18 68.58)
 		)
 		(stroke
@@
 	(wire
 		(pts
+			(xy 191.77 106.68) (xy 191.77 115.57)
+		)
+		(stroke
+			(width 0)
+			(type default)
+		)
+	)
+	(wire
+		(pts
 			(xy 43.18 120.65) (xy 49.53 120.65)
 		)
@@
 	(wire
 		(pts
-			(xy 209.55 125.73) (xy 223.52 125.73)
-		)
-		(stroke
-			(width 0)
-			(type default)
-		)
-	)
-	(wire
-		(pts
 			(xy 152.4 133.35) (xy 157.48 133.35)
 		)
@@
 	(wire
 		(pts
+			(xy 191.77 101.6) (xy 191.77 106.68)
+		)
+		(stroke
+			(width 0)
+			(type default)
+		)
+	)
+	(wire
+		(pts
 			(xy 43.18 80.01) (xy 62.23 80.01)
 		)
@@
 	)
 	(label "v_5v"
-		(at 191.77 115.57 0)
+		(at 191.77 101.6 0)
 		(effects
 			(font
@@
 			)
 		)
-		(property "Footprint" ""
+		(property "Footprint" "Resistor_SMD:R_0805_2012Metric_Pad1.20x1.40mm_HandSolder"
 			(at 155.702 154.94 90)
 			(hide yes)
@@
 			)
 		)
-		(property "Footprint" ""
+		(property "Footprint" "Capacitor_SMD:C_0805_2012Metric_Pad1.18x1.45mm_HandSolder"
 			(at 271.4752 123.19 0)
 			(hide yes)
@@
 		(lib_id "Power_Protection:USBLC6-2SC6")
 		(at 54.61 120.65 0)
+		(mirror y)
 		(unit 1)
 		(body_style 1)
@@
 		(dnp no)
 		(property "Reference" "U6"
-			(at 55.372 116.332 0)
+			(at 53.848 116.332 0)
 			(show_name no)
 			(do_not_autoplace no)
@@
 		)
 		(property "Value" "USBLC6-2SC6"
-			(at 39.37 128.524 0)
+			(at 69.85 128.524 0)
 			(show_name no)
 			(do_not_autoplace no)
@@
 		)
 		(property "Footprint" "Package_TO_SOT_SMD:SOT-23-6"
-			(at 55.88 127 0)
+			(at 53.34 127 0)
 			(hide yes)
 			(show_name no)
@@
 		)
 		(property "Datasheet" "https://www.st.com/resource/en/datasheet/usblc6-2.pdf"
-			(at 55.88 128.905 0)
+			(at 53.34 128.905 0)
 			(hide yes)
 			(show_name no)
@@
 			)
 		)
-		(property "Footprint" ""
+		(property "Footprint" "Capacitor_SMD:C_0805_2012Metric_Pad1.18x1.45mm_HandSolder"
 			(at 220.6752 123.19 0)
 			(hide yes)
@@
 	(symbol
 		(lib_id "Device:R")
-		(at 33.02 170.18 90)
+		(at 64.77 120.65 90)
 		(unit 1)
 		(body_style 1)
@@
 		(in_pos_files yes)
 		(dnp no)
-		(fields_autoplaced yes)
-		(property "Reference" "R15"
-			(at 33.02 163.83 90)
+		(property "Reference" "R4"
+			(at 64.77 118.618 90)
 			(show_name no)
 			(do_not_autoplace no)
@@
 			)
 		)
-		(property "Value" "0"
-			(at 33.02 166.37 90)
+		(property "Value" "22"
+			(at 64.77 120.904 90)
 			(show_name no)
 			(do_not_autoplace no)
@@
 		)
 		(property "Footprint" "Resistor_SMD:R_0805_2012Metric_Pad1.20x1.40mm_HandSolder"
-			(at 33.02 171.958 90)
+			(at 64.77 122.428 90)
 			(hide yes)
 			(show_name no)
@@
 		)
 		(property "Datasheet" ""
-			(at 33.02 170.18 0)
+			(at 64.77 120.65 0)
 			(hide yes)
 			(show_name no)
@@
 		)
 		(property "Description" "Resistor"
-			(at 33.02 170.18 0)
+			(at 64.77 120.65 0)
 			(hide yes)
 			(show_name no)
@@
 			)
 		)
-		(pin "2"
-		)
 		(pin "1"
 		)
+		(pin "2"
+		)
 		(instances
 			(project "neon-beat-buzzer-pcb"
 				(path "/1aa5bb6d-1502-4465-bf5e-41cf5ab51d4a"
-					(reference "R15")
+					(reference "R4")
 					(unit 1)
 				)
@@
 	)
 	(symbol
-		(lib_id "Device:R")
-		(at 64.77 120.65 90)
+		(lib_id "power:GND")
+		(at 170.18 82.55 0)
 		(unit 1)
 		(body_style 1)
@@
 		(in_pos_files yes)
 		(dnp no)
-		(property "Reference" "R4"
-			(at 64.77 118.618 90)
+		(fields_autoplaced yes)
+		(property "Reference" "#PWR012"
+			(at 170.18 88.9 0)
+			(hide yes)
 			(show_name no)
 			(do_not_autoplace no)
@@
 			)
 		)
-		(property "Value" "22"
-			(at 64.77 120.904 90)
+		(property "Value" "GND"
+			(at 170.18 87.63 0)
 			(show_name no)
 			(do_not_autoplace no)
@@
 			)
 		)
-		(property "Footprint" "Resistor_SMD:R_0805_2012Metric_Pad1.20x1.40mm_HandSolder"
-			(at 64.77 122.428 90)
+		(property "Footprint" ""
+			(at 170.18 82.55 0)
 			(hide yes)
 			(show_name no)
@@
 		)
 		(property "Datasheet" ""
-			(at 64.77 120.65 0)
+			(at 170.18 82.55 0)
 			(hide yes)
 			(show_name no)
@@
 			)
 		)
-		(property "Description" "Resistor"
-			(at 64.77 120.65 0)
+		(property "Description" "Power symbol creates a global label with name \"GND\" , ground"
+			(at 170.18 82.55 0)
 			(hide yes)
 			(show_name no)
@@
 		(pin "1"
 		)
-		(pin "2"
-		)
 		(instances
 			(project "neon-beat-buzzer-pcb"
 				(path "/1aa5bb6d-1502-4465-bf5e-41cf5ab51d4a"
-					(reference "R4")
+					(reference "#PWR012")
 					(unit 1)
 				)
@@
 	)
 	(symbol
-		(lib_id "power:GND")
-		(at 170.18 82.55 0)
+		(lib_id "Device:C")
+		(at 196.85 110.49 0)
 		(unit 1)
 		(body_style 1)
@@
 		(dnp no)
 		(fields_autoplaced yes)
-		(property "Reference" "#PWR012"
-			(at 170.18 88.9 0)
-			(hide yes)
+		(property "Reference" "C17"
+			(at 200.66 109.2199 0)
 			(show_name no)
 			(do_not_autoplace no)
@@
 					(size 1.27 1.27)
 				)
+				(justify left)
 			)
 		)
-		(property "Value" "GND"
-			(at 170.18 87.63 0)
+		(property "Value" "0.1uF"
+			(at 200.66 111.7599 0)
 			(show_name no)
 			(do_not_autoplace no)
@@
 					(size 1.27 1.27)
 				)
+				(justify left)
 			)
 		)
-		(property "Footprint" ""
-			(at 170.18 82.55 0)
+		(property "Footprint" "Capacitor_SMD:C_0805_2012Metric_Pad1.18x1.45mm_HandSolder"
+			(at 197.8152 114.3 0)
 			(hide yes)
 			(show_name no)
@@
 		)
 		(property "Datasheet" ""
-			(at 170.18 82.55 0)
+			(at 196.85 110.49 0)
 			(hide yes)
 			(show_name no)
@@
 			)
 		)
-		(property "Description" "Power symbol creates a global label with name \"GND\" , ground"
-			(at 170.18 82.55 0)
+		(property "Description" "Unpolarized capacitor"
+			(at 196.85 110.49 0)
 			(hide yes)
 			(show_name no)
@@
 		(pin "1"
 		)
+		(pin "2"
+		)
 		(instances
 			(project "neon-beat-buzzer-pcb"
 				(path "/1aa5bb6d-1502-4465-bf5e-41cf5ab51d4a"
-					(reference "#PWR012")
+					(reference "C17")
 					(unit 1)
 				)
@@
 		(in_pos_files yes)
 		(dnp no)
-		(fields_autoplaced yes)
 		(property "Reference" "U4"
-			(at 209.55 119.3098 0)
+			(at 185.928 112.014 0)
 			(show_name no)
 			(do_not_autoplace no)
@@
 			)
 		)
-		(property "Footprint" ""
+		(property "Footprint" "Package_TO_SOT_SMD:SOT-23-5"
 			(at 196.85 125.73 0)
 			(hide yes)

Commit message: project: add routed board
- Board is now fully routed (and needs some review)
- Tooling holes are added
- Needs to complete BOM

Signed-off-by: Alexis Lothoré <alexis.lothore@gmail.com>
Parts:
- removed D1, D2: D, Diode_SMD:D_0805_2012Metric_Pad1.15x1.40mm_HandSolder, symbol Device:D
- removed D6: SMF5V0A, Diode_SMD:D_SMF, symbol Diode:SMF5V0A
- added D7, D8: D_Schottky, Diode_SMD:D_SMA, symbol Device:D_Schottky
- added H1, H2, H3, H4: (no value), MountingHole:MountingHole_3.2mm_M3_Pad_Via, symbol Mechanical:MountingHole_Pad
- added R15: 10k, Resistor_SMD:R_0402_1005Metric, symbol Device:R
- C1, C11, C14, C2, C3, C4, C5, C6, C9: footprint Capacitor_SMD:C_0805_2012Metric_Pad1.18x1.45mm_HandSolder -> Capacitor_SMD:C_0603_1608Metric
- C10, C12, C13, C15, C16, C17, C7, C8: footprint Capacitor_SMD:C_0805_2012Metric_Pad1.18x1.45mm_HandSolder -> Capacitor_SMD:C_0402_1005Metric
- R1, R12, R16, R2, R3, R4, R5, R9: footprint Resistor_SMD:R_0805_2012Metric_Pad1.20x1.40mm_HandSolder -> Resistor_SMD:R_0402_1005Metric
- R10: value 100k -> 68k; footprint Resistor_SMD:R_0805_2012Metric_Pad1.20x1.40mm_HandSolder -> Resistor_SMD:R_0603_1608Metric
- R11: value 240k -> 220k; footprint Resistor_SMD:R_0805_2012Metric_Pad1.20x1.40mm_HandSolder -> Resistor_SMD:R_0603_1608Metric
- R13, R14: footprint Resistor_SMD:R_0805_2012Metric_Pad1.20x1.40mm_HandSolder -> Resistor_SMD:R_0603_1608Metric
- R6: value 2.8k -> 1.8k; footprint Resistor_SMD:R_0805_2012Metric_Pad1.20x1.40mm_HandSolder -> Resistor_SMD:R_0603_1608Metric
- R7: value 3.3k -> 3k; footprint Resistor_SMD:R_0805_2012Metric_Pad1.20x1.40mm_HandSolder -> Resistor_SMD:R_0603_1608Metric
- R8: value 2k -> 1k; footprint Resistor_SMD:R_0805_2012Metric_Pad1.20x1.40mm_HandSolder -> Resistor_SMD:R_0402_1005Metric
Connections:
- net GND: now also H1.1, H2.1, H3.1, H4.1, R15.2
- net button: now also U1.30 (GPIO20/U0RXD); no longer U1.6 (GPIO3/ADC1_CH3)
- net switch: now also D7.2 (A)
- net v_sys: now also L1.2; no longer L1.1
- net v_usb: now also D8.2 (A)
- net at R3.1: now also U6.4 (I/O2); no longer U6.3 (I/O2)
- net at U3.3 (ON): now also D7.1 (K), D8.1 (K), R15.1
- net at J4.A6 (D+), J4.B6 (D+): now also U6.3 (I/O2); no longer U6.4 (I/O2)
- net at J4.A7 (D-), J4.B7 (D-): now also U6.1 (I/O1); no longer U6.6 (I/O1)
- net at U5.5 (SW): now also L1.1; no longer L1.2
- net at R4.1: now also U6.6 (I/O1); no longer U6.1 (I/O1)
Other:
- note added: "Mounting holes"
- moved on the sheet: L1
